Commit message: connecting phase 2 and 1

File: ros2_ws/src/force_tool_planning_ros/urdf/planar_tool_arm.urdf.xacro (robot description, xacro)
@@ -140,3 +140,28 @@
     <origin xyz="0 0 0" rpy="0 0 0"/>
   </joint>
+  <!-- Position-only mock hardware for later ros2_control trajectory execution. -->
+  <ros2_control name="PlanarToolArmSystem" type="system">
+    <hardware>
+      <plugin>mock_components/GenericSystem</plugin>
+      <param name="state_following_offset">0.0</param>
+    </hardware>
+    <joint name="joint1">
+      <command_interface name="position"/>
+      <state_interface name="position">
+        <param name="initial_value">0.0</param>
+      </state_interface>
+    </joint>
+    <joint name="joint2">
+      <command_interface name="position"/>
+      <state_interface name="position">
+        <param name="initial_value">0.0</param>
+      </state_interface>
+    </joint>
+    <joint name="joint3">
+      <command_interface name="position"/>
+      <state_interface name="position">
+        <param name="initial_value">0.0</param>
+      </state_interface>
+    </joint>
+  </ros2_control>
 </robot>

Commit message: phase 2 nearly completed, also updated license

File: ros2_ws/src/force_tool_planning_ros/urdf/planar_tool_arm.urdf.xacro (robot description, xacro)
@@ -9,7 +9,13 @@
   <xacro:property name="joint_radius" value="0.075"/>
   <xacro:property name="joint_height" value="0.12"/>
-  <!-- Inverse of the selected force-aware short_inline tool_T_ee [-0.20, 0, 0]. -->
-  <xacro:property name="ee_to_tool_x" value="0.20"/>
-  <xacro:property name="tool_body_length" value="0.20"/>
+  <!-- Defaults are the inverse of force-aware short_inline tool_T_ee. -->
+  <xacro:arg name="ee_to_tool_x" default="0.20"/>
+  <xacro:arg name="ee_to_tool_y" default="0.0"/>
+  <xacro:arg name="ee_to_tool_yaw" default="0.0"/>
+  <xacro:arg name="tool_body_length" default="0.20"/>
+  <xacro:property name="ee_to_tool_x" value="$(arg ee_to_tool_x)"/>
+  <xacro:property name="ee_to_tool_y" value="$(arg ee_to_tool_y)"/>
+  <xacro:property name="ee_to_tool_yaw" value="$(arg ee_to_tool_yaw)"/>
+  <xacro:property name="tool_body_length" value="$(arg tool_body_length)"/>
   <material name="base_blue">
     <color rgba="0.12 0.35 0.65 1.0"/>
@@ -132,5 +138,6 @@
     <parent link="ee_link"/>
     <child link="tool_link"/>
-    <origin xyz="${ee_to_tool_x} 0 0" rpy="0 0 0"/>
+    <origin xyz="${ee_to_tool_x} ${ee_to_tool_y} 0"
+            rpy="0 0 ${ee_to_tool_yaw}"/>
   </joint>
   <!-- Phase 1 explicitly treats the tool frame and tool-tip frame as equal. -->
